File: kp_gmapkeyboard.kicad_pcb (KiCad board)
At the start: 12 copper layers, 20 parts, among them SW0 Encoder, SW1 Encoder, SW2 Encoder, SW3 Encoder, SW4 Encoder, U0 Teensy3.6, U1 MCP23017_SP

Commit message: fix sda/scl pins + update teensy3.6 symbol
Connections:
- U0 pad 1: Net-(U0-Pad1) -> (no net)
- U0 pad 10: Net-(U0-Pad10) -> (no net)
- U0 pad 11: Net-(U0-Pad11) -> (no net)
- U0 pad 12: Net-(U0-Pad12) -> (no net)
- U0 pad 13: Net-(U0-Pad13) -> (no net)
- U0 pad 14: Net-(U0-Pad14) -> (no net)
- U0 pad 15: Net-(U0-Pad15) -> (no net)
- U0 pad 16: Net-(U0-Pad16) -> (no net)
- U0 pad 17: Net-(U0-Pad17) -> (no net)
- U0 pad 18: sda -> (no net)
- U0 pad 19: scl -> (no net)
- U0 pad 2: Net-(U0-Pad2) -> (no net)
- U0 pad 20: Net-(U0-Pad20) -> (no net)
- U0 pad 21: Net-(U0-Pad21) -> (no net)
- U0 pad 22: Net-(U0-Pad22) -> (no net)
- U0 pad 23: Net-(U0-Pad23) -> (no net)
- U0 pad 24: Net-(U0-Pad24) -> (no net)
- U0 pad 25: Net-(U0-Pad25) -> (no net)
- U0 pad 26: Net-(U0-Pad26) -> (no net)
- U0 pad 27: Net-(U0-Pad27) -> (no net)
- U0 pad 28: Net-(U0-Pad28) -> (no net)
- U0 pad 29: Net-(U0-Pad29) -> (no net)
- U0 pad 3: Net-(U0-Pad3) -> (no net)
- U0 pad 30: Net-(U0-Pad30) -> (no net)
- U0 pad 31: Net-(U0-Pad31) -> (no net)
- U0 pad 32: Net-(U0-Pad32) -> (no net)
- U0 pad 33: Net-(U0-Pad33) -> (no net)
- U0 pad 34: Net-(U0-Pad34) -> (no net)
- U0 pad 35: Net-(U0-Pad35) -> (no net)
- U0 pad 36: Net-(U0-Pad36) -> (no net)
- U0 pad 37: Net-(U0-Pad37) -> (no net)
- U0 pad 38: Net-(U0-Pad38) -> (no net)
- U0 pad 4: Net-(U0-Pad4) -> (no net)
- U0 pad 40: Net-(U0-Pad40) -> (no net)
- U0 pad 41: Net-(U0-Pad41) -> (no net)
- U0 pad 42: Net-(U0-Pad42) -> (no net)
- U0 pad 43: Net-(U0-Pad43) -> (no net)
- U0 pad 44: Net-(U0-Pad44) -> (no net)
- U0 pad 45: Net-(U0-Pad45) -> sda
- U0 pad 46: Net-(U0-Pad46) -> scl
- U0 pad 47: Net-(U0-Pad47) -> (no net)
- U0 pad 48: Net-(U0-Pad48) -> (no net)
- U0 pad 49: Net-(U0-Pad49) -> (no net)
- U0 pad 5: Net-(U0-Pad5) -> (no net)
- U0 pad 50: Net-(U0-Pad50) -> (no net)
- U0 pad 53: Net-(U0-Pad53) -> (no net)
- U0 pad 54: Net-(U0-Pad54) -> (no net)
- U0 pad 55: Net-(U0-Pad55) -> (no net)
- U0 pad 56: Net-(U0-Pad56) -> (no net)
- U0 pad 57: Net-(U0-Pad57) -> (no net)
- U0 pad 58: Net-(U0-Pad58) -> (no net)
- U0 pad 59: Net-(U0-Pad59) -> (no net)
- U0 pad 6: Net-(U0-Pad6) -> (no net)
- U0 pad 60: Net-(U0-Pad60) -> (no net)
- U0 pad 61: Net-(U0-Pad61) -> (no net)
- U0 pad 62: Net-(U0-Pad62) -> (no net)
- U0 pad 63: Net-(U0-Pad63) -> (no net)
- U0 pad 64: Net-(U0-Pad64) -> (no net)
- U0 pad 65: Net-(U0-Pad65) -> (no net)
- U0 pad 66: Net-(U0-Pad66) -> (no net)
- U0 pad 67: Net-(U0-Pad67) -> (no net)
- U0 pad 68: Net-(U0-Pad68) -> (no net)
- U0 pad 69: Net-(U0-Pad69) -> (no net)
- U0 pad 7: Net-(U0-Pad7) -> (no net)
- U0 pad 70: Net-(U0-Pad70) -> (no net)
- U0 pad 71: Net-(U0-Pad71) -> (no net)
- U0 pad 72: Net-(U0-Pad72) -> (no net)
- U0 pad 73: Net-(U0-Pad73) -> (no net)
- U0 pad 74: Net-(U0-Pad74) -> (no net)
- U0 pad 75: Net-(U0-Pad75) -> (no net)
- U0 pad 76: Net-(U0-Pad76) -> (no net)
- U0 pad 77: Net-(U0-Pad77) -> (no net)
- U0 pad 78: Net-(U0-Pad78) -> (no net)
- U0 pad 79: Net-(U0-Pad79) -> (no net)
- U0 pad 8: Net-(U0-Pad8) -> (no net)
- U0 pad 80: Net-(U0-Pad80) -> (no net)
- U0 pad 81: Net-(U0-Pad81) -> (no net)
- U0 pad 82: Net-(U0-Pad82) -> (no net)
- U0 pad 83: Net-(U0-Pad83) -> (no net)
- U0 pad 84: Net-(U0-Pad84) -> (no net)
- U0 pad 85: Net-(U0-Pad85) -> (no net)
- U0 pad 86: Net-(U0-Pad86) -> (no net)
- U0 pad 9: Net-(U0-Pad9) -> (no net)
- U1 pad 11: Net-(U1-Pad11) -> (no net)
- U1 pad 14: Net-(U1-Pad14) -> (no net)
- U1 pad 19: Net-(U1-Pad19) -> (no net)
- U1 pad 20: Net-(U1-Pad20) -> (no net)
- U1 pad 8: Net-(U1-Pad8) -> (no net)
Routing:
- net scl: track 68.2 -> 150.7 mm
- net sda: track 75.6 -> 152.9 mm

Commit message: fix encoders pin order
when moving CW, the first pin "hit" by the turn is the lower pin number
Connections:
- C0 pad 1: pot0_rot0 -> pot0_rot1
- C1 pad 2: pot0_rot1 -> pot0_rot0
- C2 pad 1: pot1_rot0 -> pot1_rot1
- C3 pad 2: pot1_rot1 -> pot1_rot0
- C4 pad 1: pot2_rot0 -> pot2_rot1
- C5 pad 2: pot2_rot1 -> pot2_rot0
- C6 pad 1: pot3_rot0 -> pot3_rot1
- C7 pad 2: pot3_rot1 -> pot3_rot0
- C8 pad 1: pot4_rot0 -> pot4_rot1
- C9 pad 2: pot4_rot1 -> pot4_rot0
- SW0 pad A: pot0_rot0 -> pot0_rot1
- SW0 pad B: pot0_rot1 -> pot0_rot0
- SW1 pad A: pot1_rot0 -> pot1_rot1
- SW1 pad B: pot1_rot1 -> pot1_rot0
- SW2 pad A: pot2_rot0 -> pot2_rot1
- SW2 pad B: pot2_rot1 -> pot2_rot0
- SW3 pad A: pot3_rot0 -> pot3_rot1
- SW3 pad B: pot3_rot1 -> pot3_rot0
- SW4 pad A: pot4_rot0 -> pot4_rot1
- SW4 pad B: pot4_rot1 -> pot4_rot0
Routing:
- net pot3_rot0: track 78.5 -> 109.5 mm
- net pot0_rot0: track 170.2 -> 196.9 mm
- net pot1_rot0: track 137.4 -> 162.9 mm
- net pot4_rot0: track 73.2 -> 98.0 mm
- net pot2_rot0: track 105.4 -> 129.9 mm
- net pot3_rot1: track 77.5 -> 82.4 mm
- net pot0_rot1: track 161.5 -> 158.5 mm
- net pot1_rot1: track 100.9 -> 102.9 mm
- net pot2_rot1: track 82.8 -> 84.8 mm
- net pot4_rot1: track 72.2 -> 74.3 mm

Commit message: disconnect push buttons, reorder connections to match real life
Parts:
- SW0, SW1, SW2, SW3, SW4: moved to B.Cu
- moved SW4 168.7 mm to (269.2, 31.8)
- moved SW3 155.5 mm to (224.8, 17.8), turned to 270 degrees
- moved SW2 142.7 mm to (196.8, 29.2)
- moved C0 142.0 mm to (162.6, 50.8), turned to 270 degrees
- moved C1 134.1 mm to (160.0, 53.3), turned to 90 degrees
- moved C2 130.9 mm to (170.2, 50.8), turned to 270 degrees
- moved C4 128.8 mm to (175.3, 33.0), turned to 90 degrees
- moved C3 123.1 mm to (167.6, 53.3), turned to 90 degrees
- moved C5 112.3 mm to (175.3, 53.3), turned to 90 degrees
- moved C7 109.5 mm to (170.2, 30.5), turned to 270 degrees
- moved C6 109.1 mm to (167.6, 33.0), turned to 90 degrees
- moved SW1 101.1 mm to (113.0, 24.1), turned to 0 degrees
- moved SW0 95.0 mm to (24.1, 15.2), turned to 270 degrees
- moved C9 94.9 mm to (162.6, 30.5), turned to 270 degrees
- moved C8 93.7 mm to (160.0, 33.0), turned to 90 degrees
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Connections:
- SW0 pad S1: agnd -> (no net)
- SW0 pad S2: pot0_push -> (no net)
- SW1 pad S1: agnd -> (no net)
- SW1 pad S2: pot1_push -> (no net)
- SW2 pad S1: agnd -> (no net)
- SW2 pad S2: pot2_push -> (no net)
- SW3 pad S1: agnd -> (no net)
- SW3 pad S2: pot3_push -> (no net)
- SW4 pad S1: agnd -> (no net)
- SW4 pad S2: pot4_push -> (no net)
- U1 pad 2: pot3_push -> (no net)
- U1 pad 21: pot0_push -> (no net)
- U1 pad 24: pot1_push -> (no net)
- U1 pad 27: pot2_push -> (no net)
- U1 pad 5: pot4_push -> (no net)
Routing:
- net pot0_push: track 116.7 -> 0.00 mm
- net pot2_rot0: track 129.9 -> 35.1 mm
- net pot1_rot0: track 162.9 -> 71.5 mm
- net pot1_push: track 90.3 -> 0.00 mm
- net pot2_push: track 70.8 -> 0.00 mm
- net scl: track 150.7 -> 82.7 mm
- net sda: track 152.9 -> 89.0 mm
- net pot0_rot1: track 158.5 -> 221.5 mm
- net pot3_push: track 54.8 -> 0.00 mm
- net pot2_rot1: track 84.8 -> 30.4 mm
- net agnd: track 446.3 -> 499.9 mm
- net 3.3v: track 163.3 -> 113.6 mm
- net pot4_push: track 49.5 -> 0.00 mm
- net pot4_rot0: track 98.0 -> 142.6 mm
- net pot4_rot1: track 74.3 -> 118.2 mm
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
Commit message: update for kicad 7
Parts:
- SW0, SW1, SW2, SW3, SW4: value Encoder -> RotaryEncoder_Switch
Connections:
- SW0 pad S1: (no net) -> unconnected-(SW0-PadS1)
- SW0 pad S2: (no net) -> unconnected-(SW0-PadS2)
- SW1 pad S1: (no net) -> unconnected-(SW1-PadS1)
- SW1 pad S2: (no net) -> unconnected-(SW1-PadS2)
- SW2 pad S1: (no net) -> unconnected-(SW2-PadS1)
- SW2 pad S2: (no net) -> unconnected-(SW2-PadS2)
- SW3 pad S1: (no net) -> unconnected-(SW3-PadS1)
- SW3 pad S2: (no net) -> unconnected-(SW3-PadS2)
- SW4 pad S1: (no net) -> unconnected-(SW4-PadS1)
- SW4 pad S2: (no net) -> unconnected-(SW4-PadS2)
- U0 pad 1: (no net) -> unconnected-(U0-GND-Pad1)
- U0 pad 10: (no net) -> unconnected-(U0-8_TX3_MISO0_SDA0-Pad10)
- U0 pad 11: (no net) -> unconnected-(U0-9_PWM_RX2_CS0-Pad11)
- U0 pad 12: (no net) -> unconnected-(U0-10_PWM_TX2_CS0-Pad12)
- U0 pad 13: (no net) -> unconnected-(U0-11_MOSI0-Pad13)
- U0 pad 14: (no net) -> unconnected-(U0-12_MISO0-Pad14)
- U0 pad 15: (no net) -> unconnected-(U0-3.3V-Pad15)
- U0 pad 16: (no net) -> unconnected-(U0-24-Pad16)
- U0 pad 17: (no net) -> unconnected-(U0-25-Pad17)
- U0 pad 18: (no net) -> unconnected-(U0-26_TX1-Pad18)
- U0 pad 19: (no net) -> unconnected-(U0-27_RX1-Pad19)
- U0 pad 2: (no net) -> unconnected-(U0-0_RX1_MOSI1_TOUCH-Pad2)
- U0 pad 20: (no net) -> unconnected-(U0-28-Pad20)
- U0 pad 21: (no net) -> unconnected-(U0-29_PWM_CAN0TX_TOUCH-Pad21)
- U0 pad 22: (no net) -> unconnected-(U0-30_PWM_CAN0RX_TOUCH-Pad22)
- U0 pad 23: (no net) -> unconnected-(U0-31_A12_RX4_CS1-Pad23)
- U0 pad 24: (no net) -> unconnected-(U0-32_A13_TX4_SCK1-Pad24)
- U0 pad 25: (no net) -> unconnected-(U0-VBAT-Pad25)
- U0 pad 26: (no net) -> unconnected-(U0-3V3-Pad26)
- U0 pad 27: (no net) -> unconnected-(U0-GND-Pad27)
- U0 pad 28: (no net) -> unconnected-(U0-PROGRAM-Pad28)
- U0 pad 29: (no net) -> unconnected-(U0-RESET-Pad29)
- U0 pad 3: (no net) -> unconnected-(U0-1_TX1_MISO1_TOUCH-Pad3)
- U0 pad 30: (no net) -> unconnected-(U0-33_A14_TX5_CAN1TX_SCL0-Pad30)
- U0 pad 31: (no net) -> unconnected-(U0-34_A15_RX5_CAN1RX_SDA0-Pad31)
- U0 pad 32: (no net) -> unconnected-(U0-35_A16_PWM-Pad32)
- U0 pad 33: (no net) -> unconnected-(U0-36_A17_PWM-Pad33)
- U0 pad 34: (no net) -> unconnected-(U0-37_A18_PWM_SCL1-Pad34)
- U0 pad 35: (no net) -> unconnected-(U0-38_A19_PWM_SDA1-Pad35)
- U0 pad 36: (no net) -> unconnected-(U0-39_A20-Pad36)
- U0 pad 37: (no net) -> unconnected-(U0-A21_DAC0-Pad37)
- U0 pad 38: (no net) -> unconnected-(U0-A22_DAC1-Pad38)
- U0 pad 4: (no net) -> unconnected-(U0-2_PWM-Pad4)
- U0 pad 40: (no net) -> unconnected-(U0-13_SCK0_LED-Pad40)
- U0 pad 41: (no net) -> unconnected-(U0-14_A0_PWM_SCK0-Pad41)
- U0 pad 42: (no net) -> unconnected-(U0-15_A1_CS0_TOUCH-Pad42)
- U0 pad 43: (no net) -> unconnected-(U0-16_A2_SCL0_TOUCH-Pad43)
- U0 pad 44: (no net) -> unconnected-(U0-17_A3_SDA0_TOUCH-Pad44)
- U0 pad 47: (no net) -> unconnected-(U0-20_A6_PWM_CS0_SCK1-Pad47)
- U0 pad 48: (no net) -> unconnected-(U0-21_A7_PWM_CS0_SCK1-Pad48)
- U0 pad 49: (no net) -> unconnected-(U0-22_A8_PWM_TOUCH-Pad49)
- U0 pad 5: (no net) -> unconnected-(U0-3_PWM_CAN0TX_SCL2-Pad5)
- U0 pad 50: (no net) -> unconnected-(U0-23_A9_PWM_TOUCH-Pad50)
- U0 pad 53: (no net) -> unconnected-(U0-VIN-Pad53)
- U0 pad 54: (no net) -> unconnected-(U0-VUSB-Pad54)
- U0 pad 55: (no net) -> unconnected-(U0-AREF-Pad55)
- U0 pad 56: (no net) -> unconnected-(U0-A10-Pad56)
- U0 pad 57: (no net) -> unconnected-(U0-A11-Pad57)
- U0 pad 58: (no net) -> unconnected-(U0-5V-Pad58)
- U0 pad 59: (no net) -> unconnected-(U0-A26_D--Pad59)
- U0 pad 6: (no net) -> unconnected-(U0-4_PWM_CAN0RX_SDA2-Pad6)
- U0 pad 60: (no net) -> unconnected-(U0-A25_D+-Pad60)
- U0 pad 61: (no net) -> unconnected-(U0-GND-Pad61)
- U0 pad 62: (no net) -> unconnected-(U0-GND-Pad62)
- U0 pad 7: (no net) -> unconnected-(U0-5_PWM_TX1_MISO1-Pad7)
- U0 pad 8: (no net) -> unconnected-(U0-6_PWM-Pad8)
- U0 pad 9: (no net) -> unconnected-(U0-7_RX3_MISO0_SCL0-Pad9)
- U1 pad 11: (no net) -> unconnected-(U1-NC-Pad11)
- U1 pad 14: (no net) -> unconnected-(U1-NC-Pad14)
- U1 pad 19: (no net) -> unconnected-(U1-INTB-Pad19)
- U1 pad 2: (no net) -> pot3_push
- U1 pad 20: (no net) -> unconnected-(U1-INTA-Pad20)
- U1 pad 21: (no net) -> pot0_push
- U1 pad 24: (no net) -> pot1_push
- U1 pad 27: (no net) -> pot2_push
- U1 pad 5: (no net) -> pot4_push
- U1 pad 8: (no net) -> unconnected-(U1-GPB7-Pad8)
Other:
- net class Default removed
